File: KiCAD files/system/system/system.kicad_pcb (KiCad board)
At the start: 2 copper layers, 58.4 x 50.8 mm, 8 parts, among them J1 Input, SW1 SW_Push, U1 ATmega328P-P, Y1 Crystal

Commit message: Edited system schematics
Parts:
- added R2: 5.1kR, Resistor_THT:R_Axial_DIN0207_L6.3mm_D2.5mm_P10.16mm_Horizontal, F.Cu at (96.5, 66.0)
- added R3: 10kR, Resistor_THT:R_Axial_DIN0207_L6.3mm_D2.5mm_P10.16mm_Horizontal, F.Cu at (106.7, 62.0)
Connections:
- C1 pad 1: +5V -> +3.3V
- R1 pad 2: +5V -> +3.3V
- U1 pad 20: +5V -> +3.3V
- U1 pad 7: +5V -> +3.3V
Routing:
- net +3.3V: track 0.00 -> 53.2 mm
- net +5V: track 50.6 -> 8.67 mm
- net Net-(C2-Pad1): track 16.5 -> 27.6 mm
- net Net-(C3-Pad1): track 18.4 -> 18.9 mm
