File: KiCAD files/system/system/system.kicad_sch (KiCad schematic)
At the start: 8 parts, among them J1 Input, SW1 SW_Push, U1 ATmega328P-P, Y1 Crystal

Commit message: Edited system schematics
Parts:
- added R2: 5.1kR, Resistor_THT:R_Axial_DIN0207_L6.3mm_D2.5mm_P10.16mm_Horizontal, symbol Device:R
- added R3: 10kR, Resistor_THT:R_Axial_DIN0207_L6.3mm_D2.5mm_P10.16mm_Horizontal, symbol Device:R
Connections:
- net +5V: now also R2.1; no longer C1.1, R1.2, U1.20 (AVCC), U1.7 (VCC)
- net GND: now also R3.2
- new net +3.3V: C1.1, R1.2, R2.2, R3.1, U1.20 (AVCC), U1.7 (VCC)
Other:
- moved on the sheet: J1
