File: KiCAD files/system/system.kicad_pcb (KiCad board)
At the start: 2 copper layers, 14 parts, among them J1 Input, J2 Conn_01x04_Female, SW1 SW_Push, U1 ATmega328P-P, Y1 Crystal

Commit message: edited the system side circuit
Routing:
- net Net-(D1-Pad2): track 0.00 -> 18.4 mm
- net GND: track 0.00 -> 14.6 mm
- net Net-(D2-Pad2): track 0.00 -> 13.2 mm
- added copper zone on B.Cu, net GND
Other:
- board outline added: 104.1 x 61 mm
Changed lines of the file:
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@@
     )
   )
+  (gr_rect (start 86.36 53.34) (end 190.5 114.3) (layer "Edge.Cuts") (width 0.1) (fill none))
   (segment (start 99.06 73.66) (end 111.55 73.66) (width 1) (layer "B.Cu") (net 1))
   (segment (start 130.260225 83.65) (end 135.340225 88.73) (width 1) (layer "B.Cu") (net 1))
@@
   (segment (start 142.53662 86.5725) (end 137.497725 86.5725) (width 1) (layer "B.Cu") (net 1))
   (segment (start 111.55 73.66) (end 117.730225 73.66) (width 1) (layer "B.Cu") (net 1))
+  (segment (start 103.76 83.44) (end 111.71 83.44) (width 1) (layer "B.Cu") (net 2))
+  (segment (start 99.06 78.74) (end 103.76 83.44) (width 1) (layer "B.Cu") (net 2))
   (segment (start 116.84 88.9) (end 116.84 83.57) (width 1) (layer "B.Cu") (net 3))
   (segment (start 127.550225 88.9) (end 127.720225 88.73) (width 1) (layer "B.Cu") (net 3))
   (segment (start 116.84 88.9) (end 127.550225 88.9) (width 1) (layer "B.Cu") (net 3))
   (segment (start 116.84 83.57) (end 116.71 83.44) (width 1) (layer "B.Cu") (net 3))
+  (segment (start 116.13 100.07) (end 116.13 94.69) (width 1) (layer "B.Cu") (net 4))
   (segment (start 124.46 93.98) (end 127.17 91.27) (width 1) (layer "B.Cu") (net 4))
+  (segment (start 116.13 94.69) (end 116.84 93.98) (width 1) (layer "B.Cu") (net 4))
   (segment (start 116.84 93.98) (end 124.46 93.98) (width 1) (layer "B.Cu") (net 4))
   (segment (start 127.17 91.27) (end 127.720225 91.27) (width 1) (layer "B.Cu") (net 4))
-  (segment (start 116.84 99.36) (end 116.13 100.07) (width 1) (layer "B.Cu") (net 4))
-  (segment (start 116.84 93.98) (end 116.84 99.36) (width 1) (layer "B.Cu") (net 4))
   (segment (start 111.55 63.5) (end 116.84 63.5) (width 1) (layer "B.Cu") (net 5))
   (segment (start 123.035789 63.725564) (end 127.720225 68.41) (width 1) (layer "B.Cu") (net 5))
@@
   (segment (start 116.84 63.5) (end 117.065564 63.725564) (width 1) (layer "B.Cu") (net 5))
   (segment (start 122.63 63.725564) (end 123.035789 63.725564) (width 1) (layer "B.Cu") (net 5))
+  (segment (start 179.283998 68.553998) (end 175.26 64.53) (width 1) (layer "B.Cu") (net 32))
+  (segment (start 179.283998 81.28) (end 179.283998 68.553998) (width 1) (layer "B.Cu") (net 32))
+  (segment (start 171.625 72.215) (end 175.26 68.58) (width 1) (layer "B.Cu") (net 33))
+  (segment (start 171.625 80.31) (end 171.625 72.215) (width 1) (layer "B.Cu") (net 33))
+  (zone (net 2) (net_name "GND") (layer "B.Cu") (hatch edge 0.508)
+    (connect_pads (clearance 0))
+    (min_thickness 0.254) (filled_areas_thickness no)
+    (fill (thermal_gap 0.508) (thermal_bridge_width 0.508))
+    (polygon
+      (pts
+        (xy 190.5 114.3)
+        (xy 86.36 114.3)
+        (xy 86.36 53.34)
+        (xy 190.5 53.34)
+      )
+    )
+  )
 )
