File: KiCAD files/system/system.kicad_sch (KiCad schematic)
At the start: 16 parts, among them J1 Input, J2 Conn_01x04_Female, SW1 SW_Push, U1 ATmega328P-P, Y1 Crystal

Commit message: edited system side pcb
Parts:
- gave numbers to parts that had none: 2
Connections:
- net +3.3V: now also J2.1 (Pin_1)
- net GND: now also J2.4 (Pin_4)
- net PD7: now reaches R3.1
- net PD7: now also U1.13 (PD7)
- net PD6: now reaches R2.1
- net PD6: now also U1.12 (PD6)
- net data: now reaches J2.2 (Pin_2)
- net data: now also J2.3 (Pin_3), U1.2 (PD0)
- net PB1: now reaches U1.15 (PB1)
- net PB1: now also BZ1.1 (-)
Changed lines of the file:
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@@
+    (stroke (width 0) (type default) (color 0 0 0 0))
+  )
+  (wire (pts (xy 33.02 137.16) (xy 33.02 139.7))
     (stroke (width 0) (type default) (color 0 0 0 0))
   )
@@
     (stroke (width 0) (type default) (color 0 0 0 0))
   )
+  (wire (pts (xy 40.64 134.62) (xy 30.48 134.62))
+    (stroke (width 0) (type default) (color 0 0 0 0))
+  )
   (wire (pts (xy 45.72 50.8) (xy 45.72 53.34))
     (stroke (width 0) (type default) (color 0 0 0 0))
@@
     (stroke (width 0) (type default) (color 0 0 0 0))
   )
+  (wire (pts (xy 36.83 82.55) (xy 43.18 82.55))
+    (stroke (width 0) (type default) (color 0 0 0 0))
+  )
   (wire (pts (xy 52.07 115.57) (xy 59.69 115.57))
     (stroke (width 0) (type default) (color 0 0 0 0))
@@
     (stroke (width 0) (type default) (color 0 0 0 0))
   )
+  (wire (pts (xy 107.95 105.41) (xy 111.76 105.41))
+    (stroke (width 0) (type default) (color 0 0 0 0))
+  )
+  (wire (pts (xy 107.95 120.65) (xy 113.03 120.65))
+    (stroke (width 0) (type default) (color 0 0 0 0))
+  )
+  (wire (pts (xy 30.48 134.62) (xy 30.48 133.35))
+    (stroke (width 0) (type default) (color 0 0 0 0))
+  )
   (wire (pts (xy 111.76 77.47) (xy 111.76 76.2))
     (stroke (width 0) (type default) (color 0 0 0 0))
   )
+  (wire (pts (xy 30.48 142.24) (xy 40.64 142.24))
+    (stroke (width 0) (type default) (color 0 0 0 0))
+  )
   (wire (pts (xy 137.16 100.33) (xy 143.51 100.33))
     (stroke (width 0) (type default) (color 0 0 0 0))
@@
     (stroke (width 0) (type default) (color 0 0 0 0))
   )
+  (wire (pts (xy 22.86 109.22) (xy 27.94 109.22))
+    (stroke (width 0) (type default) (color 0 0 0 0))
+  )
   (wire (pts (xy 121.92 76.2) (xy 132.08 76.2))
     (stroke (width 0) (type default) (color 0 0 0 0))
   )
+  (wire (pts (xy 40.64 137.16) (xy 33.02 137.16))
+    (stroke (width 0) (type default) (color 0 0 0 0))
+  )
   (wire (pts (xy 67.31 53.34) (xy 92.71 53.34))
     (stroke (width 0) (type default) (color 0 0 0 0))
@@
     (stroke (width 0) (type default) (color 0 0 0 0))
   )
+  (wire (pts (xy 107.95 64.77) (xy 113.03 64.77))
+    (stroke (width 0) (type default) (color 0 0 0 0))
+  )
   (wire (pts (xy 67.31 134.62) (xy 92.71 134.62))
     (stroke (width 0) (type default) (color 0 0 0 0))
@@
     (stroke (width 0) (type default) (color 0 0 0 0))
   )
+  (wire (pts (xy 27.94 118.11) (xy 22.86 118.11))
+    (stroke (width 0) (type default) (color 0 0 0 0))
+  )
+  (wire (pts (xy 107.95 123.19) (xy 113.03 123.19))
+    (stroke (width 0) (type default) (color 0 0 0 0))
+  )
   (wire (pts (xy 43.18 87.63) (xy 38.1 87.63))
     (stroke (width 0) (type default) (color 0 0 0 0))
@@
   (wire (pts (xy 45.72 109.22) (xy 52.07 109.22))
     (stroke (width 0) (type default) (color 0 0 0 0))
+  )
+  (wire (pts (xy 40.64 139.7) (xy 33.02 139.7))
+    (stroke (width 0) (type default) (color 0 0 0 0))
+  )
+  (wire (pts (xy 22.86 118.11) (xy 22.86 116.84))
+    (stroke (width 0) (type default) (color 0 0 0 0))
+  )
+  (label "data" (at 33.02 138.43 0)
+    (effects (font (size 1.27 1.27)) (justify left bottom))
+  )
+  (label "PD6" (at 113.03 120.65 0)
+    (effects (font (size 1.27 1.27)) (justify left bottom))
+  )
+  (label "PD7" (at 113.03 123.19 0)
+    (effects (font (size 1.27 1.27)) (justify left bottom))
+  )
+  (label "PB1" (at 113.03 64.77 0)
+    (effects (font (size 1.27 1.27)) (justify left bottom))
+  )
+  (label "PD6" (at 22.86 109.22 0)
+    (effects (font (size 1.27 1.27)) (justify left bottom))
+  )
+  (label "PB1" (at 36.83 82.55 0)
+    (effects (font (size 1.27 1.27)) (justify left bottom))
+  )
+  (label "PD7" (at 22.86 116.84 0)
+    (effects (font (size 1.27 1.27)) (justify left bottom))
+  )
+  (label "data" (at 111.76 105.41 0)
+    (effects (font (size 1.27 1.27)) (justify left bottom))
   )
   (symbol (lib_id "power:GND") (at 59.69 115.57 0) (unit 1)
@@
   (symbol (lib_id "power:+3.3V") (at 143.51 93.98 0) (unit 1)
     (in_bom yes) (on_board yes) (fields_autoplaced)
-    (property "Reference" "#PWR?" (id 0) (at 143.51 97.79 0)
+    (property "Reference" "#PWR0101" (id 0) (at 143.51 97.79 0)
       (effects (font (size 1.27 1.27)) hide)
     )
@@
   (symbol (lib_id "Device:R") (at 45.72 60.96 0) (unit 1)
     (in_bom yes) (on_board yes) (fields_autoplaced)
-    (property "Reference" "R?" (id 0) (at 48.26 59.6899 0)
+    (property "Reference" "R5" (id 0) (at 48.26 59.6899 0)
       (effects (font (size 1.27 1.27)) (justify left))
     )
@@
   (symbol (lib_id "Device:R") (at 45.72 46.99 0) (unit 1)
     (in_bom yes) (on_board yes) (fields_autoplaced)
-    (property "Reference" "R?" (id 0) (at 48.26 45.7199 0)
+    (property "Reference" "R4" (id 0) (at 48.26 45.7199 0)
       (effects (font (size 1.27 1.27)) (justify left))
     )
@@
     (pin "2")
   )
+  (symbol (lib_id "power:GND") (at 30.48 142.24 0) (unit 1)
+    (in_bom yes) (on_board yes) (fields_autoplaced)
+    (property "Reference" "#PWR?" (id 0) (at 30.48 148.59 0)
+      (effects (font (size 1.27 1.27)) hide)
+    )
+    (property "Value" "GND" (id 1) (at 30.48 147.32 0))
+    (property "Footprint" "" (id 2) (at 30.48 142.24 0)
+      (effects (font (size 1.27 1.27)) hide)
+    )
+    (property "Datasheet" "" (id 3) (at 30.48 142.24 0)
+      (effects (font (size 1.27 1.27)) hide)
+    )
+    (pin "1")
+  )
   (symbol (lib_id "Device:LED") (at 41.91 109.22 180) (unit 1)
     (in_bom yes) (on_board yes) (fields_autoplaced)
@@
   (symbol (lib_id "power:+3.3V") (at 58.42 53.34 0) (unit 1)
     (in_bom yes) (on_board yes) (fields_autoplaced)
-    (property "Reference" "#PWR?" (id 0) (at 58.42 57.15 0)
+    (property "Reference" "#PWR0105" (id 0) (at 58.42 57.15 0)
       (effects (font (size 1.27 1.27)) hide)
     )
@@
   (symbol (lib_id "power:+5V") (at 45.72 39.37 0) (unit 1)
     (in_bom yes) (on_board yes) (fields_autoplaced)
-    (property "Reference" "#PWR?" (id 0) (at 45.72 43.18 0)
+    (property "Reference" "#PWR0110" (id 0) (at 45.72 43.18 0)
       (effects (font (size 1.27 1.27)) hide)
     )
@@
   (symbol (lib_id "power:GND") (at 45.72 68.58 0) (unit 1)
     (in_bom yes) (on_board yes) (fields_autoplaced)
-    (property "Reference" "#PWR?" (id 0) (at 45.72 74.93 0)
+    (property "Reference" "#PWR0112" (id 0) (at 45.72 74.93 0)
       (effects (font (size 1.27 1.27)) hide)
     )
@@
   (symbol (lib_id "power:+3.3V") (at 93.98 41.91 0) (unit 1)
     (in_bom yes) (on_board yes) (fields_autoplaced)
-    (property "Reference" "#PWR?" (id 0) (at 93.98 45.72 0)
+    (property "Reference" "#PWR0111" (id 0) (at 93.98 45.72 0)
       (effects (font (size 1.27 1.27)) hide)
     )
@@
     (pin "2")
   )
+  (symbol (lib_id "power:+3.3V") (at 30.48 133.35 0) (unit 1)
+    (in_bom yes) (on_board yes) (fields_autoplaced)
+    (property "Reference" "#PWR?" (id 0) (at 30.48 137.16 0)
+      (effects (font (size 1.27 1.27)) hide)
+    )
+    (property "Value" "+3.3V" (id 1) (at 30.48 128.27 0))
+    (property "Footprint" "" (id 2) (at 30.48 133.35 0)
+      (effects (font (size 1.27 1.27)) hide)
+    )
+    (property "Datasheet" "" (id 3) (at 30.48 133.35 0)
+      (effects (font (size 1.27 1.27)) hide)
+    )
+    (pin "1")
+  )
   (symbol (lib_id "Switch:SW_Push") (at 119.38 109.22 270) (unit 1)
     (in_bom yes) (on_board yes) (fields_autoplaced)
@@
   )
   (symbol_instances
+    (path "/19c32ca3-7a65-4db2-b139-c8394a8c32b4"
+      (reference "#PWR0101") (unit 1) (value "+3.3V") (footprint "")
+    )
     (path "/7bd4950f-6eee-43e4-bd48-4b535e69d247"
       (reference "#PWR0102") (unit 1) (value "GND") (footprint "")
@@
       (reference "#PWR0104") (unit 1) (value "GND") (footprint "")
     )
+    (path "/585372d9-072e-4298-902a-dbe5a4230ce7"
+      (reference "#PWR0105") (unit 1) (value "+3.3V") (footprint "")
+    )
     (path "/ad280cdc-2c85-4211-98af-a61695a3e90c"
       (reference "#PWR0106") (unit 1) (value "+5V") (footprint "")
@@
       (reference "#PWR0109") (unit 1) (value "GND") (footprint "")
     )
-    (path "/19c32ca3-7a65-4db2-b139-c8394a8c32b4"
-      (reference "#PWR?") (unit 1) (value "+3.3V") (footprint "")
-    )
-    (path "/585372d9-072e-4298-902a-dbe5a4230ce7"
-      (reference "#PWR?") (unit 1) (value "+3.3V") (footprint "")
-    )
     (path "/66c79a79-a322-4170-a991-452ddccb89cb"
-      (reference "#PWR?") (unit 1) (value "+5V") (footprint "")
+      (reference "#PWR0110") (unit 1) (value "+5V") (footprint "")
+    )
+    (path "/9a062bae-fa39-4731-8307-4dd6a924ed50"
+      (reference "#PWR0111") (unit 1) (value "+3.3V") (footprint "")
     )
     (path "/8eaea635-237d-4aae-8265-637174364b6e"
+      (reference "#PWR0112") (unit 1) (value "GND") (footprint "")
+    )
+    (path "/314bee24-7551-4061-bacf-7c3db6d80d27"
       (reference "#PWR?") (unit 1) (value "GND") (footprint "")
     )
-    (path "/9a062bae-fa39-4731-8307-4dd6a924ed50"
+    (path "/d67820f3-633a-47b0-adb5-ff5009f3e09a"
       (reference "#PWR?") (unit 1) (value "+3.3V") (footprint "")
     )
@@
       (reference "R3") (unit 1) (value "R") (footprint "Resistor_THT:R_Axial_DIN0207_L6.3mm_D2.5mm_P10.16mm_Horizontal")
     )
+    (path "/218f3874-86de-43d1-ad93-31612cd48ff6"
+      (reference "R4") (unit 1) (value "5.1kR") (footprint "Resistor_THT:R_Axial_DIN0207_L6.3mm_D2.5mm_P10.16mm_Horizontal")
+    )
     (path "/1de8b467-ee66-4fc5-ad7d-f052303838c2"
-      (reference "R?") (unit 1) (value "10kR") (footprint "Resistor_THT:R_Axial_DIN0207_L6.3mm_D2.5mm_P10.16mm_Horizontal")
-    )
-    (path "/218f3874-86de-43d1-ad93-31612cd48ff6"
-      (reference "R?") (unit 1) (value "5.1kR") (footprint "Resistor_THT:R_Axial_DIN0207_L6.3mm_D2.5mm_P10.16mm_Horizontal")
+      (reference "R5") (unit 1) (value "10kR") (footprint "Resistor_THT:R_Axial_DIN0207_L6.3mm_D2.5mm_P10.16mm_Horizontal")
     )
     (path "/dcbe2ab9-36f3-4396-bb36-2ca532473c12"

Commit message: edited system pcb
Parts:
- removed J2: Conn_01x04_Female, Connector_PinHeader_2.54mm:PinHeader_1x04_P2.54mm_Horizontal, symbol Connector:Conn_01x04_Female
- added J2: Conn_01x06_Female, Connector_PinHeader_2.54mm:PinHeader_1x06_P2.54mm_Vertical, symbol Connector:Conn_01x06_Female
- C1: value C_Polarized -> 10u
- R1: value R -> 10k
- R2, R3: value R -> 440
Connections:
- net +5V: now also J2.2 (Pin_2)
- net GND: now also J2.3 (Pin_3)
- net PD6: now also U1.17 (PB3); no longer U1.12 (PD6)
- net PD7: now also U1.18 (PB4); no longer U1.13 (PD7)
- net rxd: now reaches U1.3 (PD1)
- net rxd: now also J2.5 (Pin_5)
- net data renamed txd
- net txd: now also J2.4 (Pin_4)
- no-connect marks 0 -> 1
Other:
- moved on the sheet: R1, SW1
